File: pre carga inteligente.kicad_sch (KiCad schematic)
At the start: 53 parts, among them J1 Screw_Terminal_01x02, J2 Screw_Terminal_01x02, K1 SANYOU_SRD_Form_C, K2 SANYOU_SRD_Form_C, Q1 NMOS, Q2 NMOS, Q3 NMOS, U1 LM393, U2 LM393

Commit message: Add boom and small symbol names corrections
Parts:
- B1: value Buck DC/DC -> Buck XL7015
- GND_IN1, GND_OUT1, Path1, Path2, Vin1, Vout1: now left out of the parts list
- K1, K2: value SANYOU_SRD_Form_C -> ICR 50.51.9.048
- Q1, Q2, Q3: value NMOS -> 75NF75
- R21: value 100K -> 4,7K
- R23: value R -> 8,2K
- R24: value R -> R10K
Changed lines of the file:
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@@
 			)
 		)
-		(property "Value" "NMOS"
+		(property "Value" "75NF75"
 			(at 162.306 43.18 0)
 			(show_name no)
@@
 			)
 		)
-		(property "Value" "100K"
+		(property "Value" "4,7K"
 			(at 121.92 76.2 0)
 			(show_name no)
@@
 			)
 		)
-		(property "Value" "Buck DC/DC"
+		(property "Value" "Buck XL7015"
 			(at 54.61 191.77 0)
 			(show_name no)
@@
 			)
 		)
-		(property "Description" ""
+		(property "Description" "Conversor buck"
 			(at 49.53 181.61 0)
 			(hide yes)
@@
 		(body_style 1)
 		(exclude_from_sim no)
-		(in_bom yes)
+		(in_bom no)
 		(on_board yes)
 		(in_pos_files yes)
@@
 			)
 		)
-		(property "Value" "NMOS"
+		(property "Value" "75NF75"
 			(at 163.83 133.3499 0)
 			(show_name no)
@@
 		(body_style 1)
 		(exclude_from_sim no)
-		(in_bom yes)
+		(in_bom no)
 		(on_board yes)
 		(in_pos_files yes)
@@
 			)
 		)
-		(property "Value" "R"
-			(at 130.048 106.934 90)
+		(property "Value" "R10K"
+			(at 132.842 106.172 90)
 			(show_name no)
 			(do_not_autoplace no)
@@
 		(body_style 1)
 		(exclude_from_sim no)
-		(in_bom yes)
+		(in_bom no)
 		(on_board yes)
 		(in_pos_files yes)
@@
 			)
 		)
-		(property "Value" "R"
-			(at 119.126 106.68 90)
+		(property "Value" "8,2K"
+			(at 121.92 106.426 90)
 			(show_name no)
 			(do_not_autoplace no)
@@
 			)
 		)
-		(property "Value" "SANYOU_SRD_Form_C"
+		(property "Value" "ICR 50.51.9.048"
 			(at 210.82 132.0799 0)
 			(show_name no)
@@
 			)
 		)
-		(property "Datasheet" "http://www.sanyourelay.ca/public/products/pdf/SRD.pdf"
+		(property "Datasheet" "https://www.icr-reles.com.br/wp-content/themes/education-zone/pdf/S5051rev.pdf"
 			(at 199.39 130.81 0)
 			(hide yes)
@@
 			)
 		)
-		(property "Description" "Sanyo SRD relay, Single Pole Miniature Power Relay,"
+		(property "Description" "rele icr 48v"
 			(at 199.39 130.81 0)
 			(hide yes)
@@
 			)
 		)
-		(property "Value" "SANYOU_SRD_Form_C"
+		(property "Value" "ICR 50.51.9.048"
 			(at 210.82 41.9099 0)
 			(show_name no)
@@
 			)
 		)
-		(property "Datasheet" "http://www.sanyourelay.ca/public/products/pdf/SRD.pdf"
+		(property "Datasheet" "https://www.icr-reles.com.br/wp-content/themes/education-zone/pdf/S5051rev.pdf"
 			(at 199.39 40.64 0)
 			(hide yes)
@@
 			)
 		)
-		(property "Description" "Sanyo SRD relay, Single Pole Miniature Power Relay,"
+		(property "Description" "rele icr 48v"
 			(at 199.39 40.64 0)
 			(hide yes)
@@
 		(body_style 1)
 		(exclude_from_sim no)
-		(in_bom yes)
+		(in_bom no)
 		(on_board yes)
 		(in_pos_files yes)
@@
 		(body_style 1)
 		(exclude_from_sim no)
-		(in_bom yes)
+		(in_bom no)
 		(on_board yes)
 		(in_pos_files yes)
@@
 		(body_style 1)
 		(exclude_from_sim no)
-		(in_bom yes)
+		(in_bom no)
 		(on_board yes)
 		(in_pos_files yes)
@@
 			)
 		)
-		(property "Value" "NMOS"
+		(property "Value" "75NF75"
 			(at 170.434 85.09 0)
 			(show_name no)
